Commit message: Integrate servo load path and RL sensor package

File: generated/urdf/zeroth01_rl_round_v1.urdf (robot description, URDF)
Before this commit: robot zeroth01_rl_round_v1_16dof, 18 links, 17 joints
Links:
- added link battery_pack, mass 0.34; visual box size=0.075 0.038 0.038
- added link camera_module, mass 0.035; visual box size=0.065 0.02 0.018
- added link camera_optical_frame
- added link compute_module, mass 0.18; visual box size=0.105 0.02 0.07
- added link imu_module, mass 0.012; visual box size=0.032 0.025 0.008
- link Torso: mass 2.45513574175 -> 2.48634993491
Joints:
- added joint battery_pack_mount: type fixed, parent Torso, child battery_pack, origin xyz=0 0 -0.044 rpy=0 0 0
- added joint camera_module_mount: type fixed, parent Torso, child camera_module, origin xyz=0 -0.03 0.108 rpy=0 0 0
- added joint camera_optical_frame_joint: type fixed, parent camera_module, child camera_optical_frame, origin xyz=0 -0.011 0 rpy=-1.57079632679 0 3.14159265359
- added joint compute_module_mount: type fixed, parent Torso, child compute_module, origin xyz=0 0.022 0.015 rpy=0 0 0
- added joint imu_module_mount: type fixed, parent Torso, child imu_module, origin xyz=0 0.008 0.01 rpy=0 0 0

Commit message: Publish minimal-cosmetic Zeroth-01 RL mechanical baseline

File: generated/urdf/zeroth01_rl_round_v1.urdf (robot description, URDF)
Before this commit: robot zeroth01_rl_round_v1_16dof, 23 links, 22 joints
Links:
- added link eye_display_module, mass 0.011; visual box size=0.0510853 0.0018615 0.0201119
- added link tof_module, mass 0.002; visual box size=0.012 0.003 0.01
- added link tof_optical_frame
- link Torso: mass 2.48634993491 -> 2.34106825776; geometry collision box size=0.046 0.068 0.056; collision box size=0.108 0.076 0.13
- link camera_module: mass 0.035 -> 0.004; geometry visual box size=0.025 0.0114 0.023862
Joints:
- added joint eye_display_module_mount: type fixed, parent Torso, child eye_display_module, origin xyz=0 -0.042 0.115 rpy=1.57079632679 0 0
- added joint tof_module_mount: type fixed, parent Torso, child tof_module, origin xyz=0.031 -0.042 0.092 rpy=1.57079632679 0 0
- added joint tof_optical_frame_joint: type fixed, parent tof_module, child tof_optical_frame, origin xyz=0 -0.002 0 rpy=-1.57079632679 0 3.14159265359
- joint camera_module_mount: origin xyz=0 -0.03 0.108 rpy=0 0 0 -> xyz=0 -0.04 0.091 rpy=-1.57079632679 0 0
- joint camera_optical_frame_joint: origin xyz=0 -0.011 0 rpy=-1.57079632679 0 3.14159265359 -> xyz=0 -0.007 0 rpy=-1.57079632679 0 3.14159265359

Commit message: Publish Round V3 ears rounded arms and chibi hands

File: generated/urdf/zeroth01_rl_round_v1.urdf (robot description, URDF)
Before this commit: robot zeroth01_rl_round_v1_16dof, 26 links, 25 joints
Links:
- link Left_Hand: mass 0.075184887 -> 0.186513252268; geometry collision box size=0.046 0.049 0.06; collision mesh filename=meshes/Left_Hand.stl
- link Torso: mass 2.34106825776 -> 2.34054437788; geometry collision box size=0.046 0.068 0.056; collision box size=0.108 0.076 0.13
- link eye_display_module: mass 0.011 -> 0.129; geometry visual box size=0.1055 0.008 0.0672
- link hand_right: mass 0.075183656 -> 0.18651364859; geometry collision box size=0.046 0.049 0.06; collision mesh filename=meshes/hand_right.stl
- link left_shoulder_yaw_motor: mass 0.171459652 -> 0.206635158636; geometry collision box size=0.07 0.046 0.057; collision mesh filename=meshes/left_shoulder_yaw_motor.stl
- link right_shoulder_yaw_motor: mass 0.17145988099999998 -> 0.206635387636; geometry collision box size=0.07 0.046 0.057; collision mesh filename=meshes/right_shoulder_yaw_motor.stl
Joints:
- joint camera_module_mount: origin xyz=0 -0.04 0.091 rpy=-1.57079632679 0 0 -> xyz=0 -0.03 0.151 rpy=-1.57079632679 0 0
- joint eye_display_module_mount: origin xyz=0 -0.042 0.115 rpy=1.57079632679 0 0 -> xyz=0 -0.025 0.105 rpy=1.57079632679 0 0
- joint tof_module_mount: origin xyz=0.031 -0.042 0.092 rpy=1.57079632679 0 0 -> xyz=0.026 -0.034 0.151 rpy=1.57079632679 0 0
