Commit message: Release v3 RL-fixed CoreS3 mechanical package

File: generated/urdf/physical_mount_v3_rl_fixed/zeroth01_physical_mount_v3_rl_fixed_18dof.urdf (robot description, URDF)
Before this commit: robot zeroth01_physical_mount_v3_rl_fixed_18dof, 41 links, 40 joints
Links:
- removed link m5stack_stackchan_k151_head_pod
- removed link stackchan_k151_torso_adapter
- added link cores3_internal_torso_cradle, mass 0.006; collision box size=0.0095 0.058 0.04; visual box size=0.0095 0.058 0.04
- added link m5stack_cores3_head_module, mass 0.0727; collision box size=0.0155 0.054 0.054; visual box size=0.001 0.046 0.046
- link FOOT: geometry collision box size=0.110059646194 0.00700011141312 0.075087498283; visual mesh filename=meshes/skeleton/FOOT.stl
- link FOOT_2: geometry collision box size=0.110059615669 0.00700008863371 0.0750874647737; visual mesh filename=meshes/skeleton/FOOT_2.stl
- link Z_BOT2_MASTER_BODY_SKELETON: geometry collision box size=0.105063672845 0.0800835889392 0.18; visual mesh filename=meshes/v3/body_skeleton_top_trimmed_45mm.stl scale=0.001 0.001 0.001
- link left_ankle_roll_carrier: geometry collision cylinder length=0.03 radius=0.014; visual mesh filename=meshes/v3/left_ankle_roll_carrier.stl scale=0.001 0.001 0.001
- link right_ankle_roll_carrier: geometry collision cylinder length=0.03 radius=0.014; visual mesh filename=meshes/v3/right_ankle_roll_carrier.stl scale=0.001 0.001 0.001
Joints:
- removed joint stackchan_head_adapter_fixed_joint
- removed joint stackchan_head_pod_fixed_joint
- added joint cores3_head_module_fixed_joint: type fixed, parent cores3_internal_torso_cradle, child m5stack_cores3_head_module, origin xyz=0.00875 0 0 rpy=0 0 0
- added joint cores3_internal_cradle_fixed_joint: type fixed, parent Z_BOT2_MASTER_BODY_SKELETON, child cores3_internal_torso_cradle, origin xyz=2.3889801322e-05 -0.029999990488 0.018 rpy=0 -0 -1.57
- joint camera_optical_frame_joint: origin xyz=0.03075 0 -0.02 rpy=0 1.57079632679 0 -> xyz=0.00825 0 -0.02 rpy=0 1.57079632679 0; parent m5stack_stackchan_k151_head_pod -> m5stack_cores3_head_module
- joint head_imu_frame_joint: parent m5stack_stackchan_k151_head_pod -> m5stack_cores3_head_module
- joint head_speaker_frame_joint: origin xyz=-0.03075 0 0 rpy=0 0 0 -> xyz=-0.00775 0 0 rpy=0 0 0; parent m5stack_stackchan_k151_head_pod -> m5stack_cores3_head_module
- joint left_ankle_roll: origin xyz=4.99999946446e-08 0.05 9.80754505386e-10 rpy=1.00916034731e-22 -1.35956678732e-19 3.54708617595e-22 -> xyz=2.99999967854e-08 0.03 5.88452703232e-10 rpy=1.00916034731e-22 -1.35956678732e-19 3.54708617595e-22
- joint left_microphone_frame_joint: origin xyz=0.03075 0.015 -0.02 rpy=0 0 0 -> xyz=0.00825 0.015 -0.02 rpy=0 0 0; parent m5stack_stackchan_k151_head_pod -> m5stack_cores3_head_module
- joint left_sole_front_lateral_contact_joint: origin xyz=-0.0449760891509 0.0270000455653 -0.0300357943822 rpy=0 0 0 -> xyz=-0.0449760911509 0.0250000455653 -0.0300357944214 rpy=0 0 0
- joint left_sole_front_medial_contact_joint: origin xyz=-0.0450238283612 0.0270000444361 0.0299641866259 rpy=0 0 0 -> xyz=-0.0450238303612 0.0250000444361 0.0299641865867 rpy=0 0 0
- joint left_sole_rear_lateral_contact_joint: origin xyz=0.0550238791959 0.0269999455637 -0.0299562290316 rpy=0 0 0 -> xyz=0.0550238771959 0.0249999455637 -0.0299562290708 rpy=0 0 0
- joint left_sole_rear_medial_contact_joint: origin xyz=0.0549761399855 0.0269999444346 0.0300437519765 rpy=0 0 0 -> xyz=0.0549761379855 0.0249999444346 0.0300437519372 rpy=0 0 0
- joint right_ankle_roll: origin xyz=1.7320515671e-08 -0.05 -3.36602488382e-08 rpy=2.65938566936e-22 1.98579295956e-19 2.70901650611e-23 -> xyz=1.03923094019e-08 -0.03 -2.01961493015e-08 rpy=2.65938566936e-22 1.98579295956e-19 2.70901650611e-23
- joint right_microphone_frame_joint: origin xyz=0.03075 -0.015 -0.02 rpy=0 0 0 -> xyz=0.00825 -0.015 -0.02 rpy=0 0 0; parent m5stack_stackchan_k151_head_pod -> m5stack_cores3_head_module
- joint right_sole_front_lateral_contact_joint: origin xyz=-0.0449761172025 -0.0270000358004 0.0300357611551 rpy=0 0 0 -> xyz=-0.0449761178953 -0.0250000358004 0.0300357625015 rpy=0 0 0
- joint right_sole_front_medial_contact_joint: origin xyz=-0.0450238356282 -0.0269999954247 -0.0299642198695 rpy=0 0 0 -> xyz=-0.0450238363211 -0.0249999954247 -0.0299642185231 rpy=0 0 0
- joint right_sole_rear_lateral_contact_joint: origin xyz=0.0550238511718 -0.0270000011059 0.0299562304455 rpy=0 0 0 -> xyz=0.055023850479 -0.0250000011059 0.0299562317919 rpy=0 0 0
- joint right_sole_rear_medial_contact_joint: origin xyz=0.0549761327461 -0.0269999607301 -0.0300437505791 rpy=0 0 0 -> xyz=0.0549761320533 -0.0249999607301 -0.0300437492327 rpy=0 0 0
