Commit message: Fix Zeroth-01 actuator load paths and remove redundant parts

File: generated/urdf/physical_mount_v4_original_minimal/zeroth01_physical_mount_v4_original_minimal_18dof.urdf (robot description, URDF)
Before this commit: robot zeroth01_physical_mount_v4_original_minimal_18dof, 39 links, 38 joints
Links:
- removed link torso_imu_frame
- removed link v4_battery_pack
- removed link v4_compute_module
- removed link v4_rear_service_pod
- removed link v4_torso_imu
- link 3215_1Flange: geometry collision cylinder length=0.0968711735038 radius=0.016; visual mesh filename=meshes/skeleton/3215_1Flange.stl
- link 3215_1Flange_2: geometry collision cylinder length=0.0968711735038 radius=0.016; visual mesh filename=meshes/skeleton/3215_1Flange_2.stl
- link 3215_BothFlange_10: geometry collision cylinder length=0.100506654506 radius=0.018; visual mesh filename=meshes/skeleton/3215_BothFlange_10.stl
- link 3215_BothFlange_13: geometry collision cylinder length=0.0820039022888 radius=0.017; visual mesh filename=meshes/v4/left_source_shin_shortened_18mm.stl scale=0.001 0.001 0.001
- link 3215_BothFlange_14: geometry collision cylinder length=0.0820060972626 radius=0.017; visual mesh filename=meshes/v4/right_source_shin_shortened_18mm.stl scale=0.001 0.001 0.001
- link 3215_BothFlange_5: geometry collision cylinder length=0.0372205588351 radius=0.015; visual mesh filename=meshes/skeleton/3215_BothFlange_5.stl
- link 3215_BothFlange_6: geometry collision cylinder length=0.0377116692815 radius=0.015; visual mesh filename=meshes/skeleton/3215_BothFlange_6.stl
- link 3215_BothFlange_9: geometry collision cylinder length=0.100506654506 radius=0.018; visual mesh filename=meshes/skeleton/3215_BothFlange_9.stl
- link FINGER_1: mass 0.016 -> 0.005; geometry 
- link FINGER_1_2: mass 0.016 -> 0.005; geometry 
- link FOOT: geometry collision box size=0.0900325993058 0.00600009077296 0.0410715959554; visual mesh filename=meshes/skeleton/FOOT.stl
- link FOOT_2: geometry collision box size=0.0900325812063 0.0060000588152 0.0410715687113; visual mesh filename=meshes/skeleton/FOOT_2.stl
- link L_ARM_MIRROR_1: geometry collision cylinder length=0.0672572919467 radius=0.014; visual mesh filename=meshes/replacements/L_ARM_MIRROR_1_WRIST_TRIMMED.stl
- link R_ARM_MIRROR_1: geometry collision cylinder length=0.0672572919467 radius=0.014; visual mesh filename=meshes/replacements/R_ARM_MIRROR_1_WRIST_TRIMMED.stl
- link U_HIP_L: geometry collision cylinder length=0.0591121814857 radius=0.012; visual mesh filename=meshes/skeleton/U_HIP_L.stl
- link U_HIP_R: geometry collision cylinder length=0.0591121814857 radius=0.012; visual mesh filename=meshes/skeleton/U_HIP_R.stl
- link Z_BOT2_MASTER_BODY_SKELETON: mass 0.728 -> 1.041; geometry collision box size=0.105063672845 0.0800835889392 0.18; visual mesh filename=meshes/v4/body_original_head_interface_trimmed_2p5mm.stl scale=0.001 0.001 0.001
- link Z_BOT2_MASTER_SHOULDER2: geometry collision cylinder length=0.0284949824531 radius=0.011; visual mesh filename=meshes/skeleton/Z_BOT2_MASTER_SHOULDER2.stl
- link Z_BOT2_MASTER_SHOULDER2_2: geometry collision cylinder length=0.0284949824531 radius=0.011; visual mesh filename=meshes/skeleton/Z_BOT2_MASTER_SHOULDER2_2.stl
- link left_ankle_roll_carrier: geometry collision cylinder length=0.0265 radius=0.014; visual mesh filename=meshes/v4/left_direct_ankle_carrier_26p5mm.stl scale=0.001 0.001 0.001
- link right_ankle_roll_carrier: geometry collision cylinder length=0.0265 radius=0.014; visual mesh filename=meshes/v4/right_direct_ankle_carrier_26p5mm.stl scale=0.001 0.001 0.001
Joints:
- removed joint torso_imu_frame_joint
- removed joint v4_battery_pack_fixed_joint
- removed joint v4_compute_module_fixed_joint
- removed joint v4_rear_service_pod_fixed_joint
- removed joint v4_torso_imu_fixed_joint
- joint left_sole_front_lateral_contact_joint: origin xyz=-0.0449760715508 0.0446000855652 -0.030035794037 rpy=0 0 0 -> xyz=-0.0449760805508 0.0356000855652 -0.0300357942135 rpy=0 0 0
- joint left_sole_front_medial_contact_joint: origin xyz=-0.0450238107612 0.0446000844361 0.0299641869711 rpy=0 0 0 -> xyz=-0.0450238197612 0.0356000844361 0.0299641867946 rpy=0 0 0
- joint left_sole_rear_lateral_contact_joint: origin xyz=0.0550238967959 0.0445999855637 -0.0299562286864 rpy=0 0 0 -> xyz=0.0550238877959 0.0355999855637 -0.0299562288629 rpy=0 0 0
- joint left_sole_rear_medial_contact_joint: origin xyz=0.0549761575856 0.0445999844346 0.0300437523217 rpy=0 0 0 -> xyz=0.0549761485856 0.0355999844346 0.0300437521451 rpy=0 0 0
- joint right_sole_front_lateral_contact_joint: origin xyz=-0.0449761111057 -0.0446000758004 0.0300357493066 rpy=0 0 0 -> xyz=-0.0449761142233 -0.0356000758004 0.0300357553655 rpy=0 0 0
- joint right_sole_front_medial_contact_joint: origin xyz=-0.0450238295314 -0.0446000354247 -0.029964231718 rpy=0 0 0 -> xyz=-0.0450238326491 -0.0356000354247 -0.0299642256591 rpy=0 0 0
- joint right_sole_rear_lateral_contact_joint: origin xyz=0.0550238572687 -0.0446000411059 0.0299562185971 rpy=0 0 0 -> xyz=0.055023854151 -0.0356000411059 0.0299562246559 rpy=0 0 0
- joint right_sole_rear_medial_contact_joint: origin xyz=0.0549761388429 -0.0446000007301 -0.0300437624275 rpy=0 0 0 -> xyz=0.0549761357252 -0.0356000007301 -0.0300437563687 rpy=0 0 0
